File: Hardware/v3 (wireless)/Mouse v3.kicad_pcb (KiCad board)
At the start: 2 copper layers, 48 x 66 mm, 21 parts, among them SW1 Scroll + Middle, U1 PMW3389, U3 XC6206-1.8V, U4 XIAO_ESP32C3

Commit message: updated pcb v3
Parts:
- moved REF** 15.0 mm to (120.0, 44.9)
- moved REF** 15.0 mm to (160.0, 44.9)
- moved S1 15.0 mm to (124.0, 54.9)
- moved S2 15.0 mm to (156.0, 54.9)
- moved SW1 15.0 mm to (132.5, 54.5)
Routing:
- net /Right Click: track 90.1 -> 108.1 mm
- net /Middle Click: track 56.9 -> 73.3 mm
- net /Rot A: track 62.4 -> 78.7 mm
- net /Left Click: track 47.4 -> 60.5 mm
- net /Rot B: track 45.3 -> 56.9 mm
- net GND: track 36.8 -> 34.5 mm, vias 35 -> 34
Other:
- board size 48 x 66 mm -> 48 x 83 mm
